File: Hardware/PCB_CAD/MuseMatrix_Core/_autosave-Column_7_Rows.kicad_sch (KiCad schematic)
At the start: 46 parts, among them J14 Conn_01x03_Pin, J15 Conn_01x07_Socket, J4 Conn_01x07_Socket, Q2 2N3904, Q3 2N3904, Q4 2N3904, Q5 2N3904, Q6 2N3904, Q7 2N3904, Q8 2N3904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

Commit message: pcb update
Parts:
- added J13: Conn_01x03_Pin, Connector_JST:JST_EH_B3B-EH-A_1x03_P2.50mm_Vertical, symbol Connector:Conn_01x03_Pin
- R28: footprint Potentiometer_THT:Potentiometer_Bourns_PTV09A-1_Single_Vertical -> Resistor_SMD:R_0402_1005Metric
- renumbered D8 to D1, J14 to J2, J15 to J3, Q9 to Q1, R29 to R1, R43 to R2
Connections:
- net +3.3V: now also J13.3 (Pin_3)
- net GND: now also J13.1 (Pin_1)
- net column_voltage: now also J13.2 (Pin_2)
