File: Hardware/PCB_CAD/MuseMatrix_Core/Main_Board.kicad_sch (KiCad schematic)
At the start: 10 parts, among them J10 Conn_01x03_Pin, J11 Conn_01x03_Pin, J12 Conn_01x03_Pin, J5 Conn_01x07_Socket, J6 Conn_01x03_Pin, J7 Conn_01x03_Pin, J8 Conn_01x03_Pin, J9 Conn_01x03_Pin, U2 74HC595, U3 74HC165

Commit message: pcb update
Parts:
- J10, J11, J12, J6, J7, J8, J9: footprint (none) -> Connector_JST:JST_EH_B3B-EH-A_1x03_P2.50mm_Vertical
- J5: footprint (none) -> Connector_JST:JST_EH_B7B-EH-A_1x07_P2.50mm_Vertical
- U2, U3: footprint (none) -> Package_SO:SOIC-16_3.9x9.9mm_P1.27mm
Connections:
- net Rst is gone; now on net +3.3V: U2.10 (~{SRCLR})
- net no_en is gone; now on net GND: U2.13 (~{OE})
- net GND: now also U2.8 (GND)
- net Parallel_Load renamed LOAD_165
- net Row_Serial_H renamed DATA_OUT_165
- net Row_Serial_L: no longer names the net of U3.7 (~{Q7})
- net Serial_Column_input renamed DATA_IN_595
- net Shift_Clock renamed clock_595
- net Storage_Clock renamed LATCH_595
- net clock1_input renamed clock_165
- no-connect marks 0 -> 1
Changed lines of the file:
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@@
 	(generator_version "8.0")
 	(paper "A4")
+	(no_connect
+		(at 116.84 54.61)
+	)
 	(hierarchical_label "jst3"
 		(shape input)
@@
 		)
 	)
-	(hierarchical_label "Serial_Column_input"
+	(hierarchical_label "DATA_IN_595"
 		(shape input)
 		(at 161.29 57.15 180)
@@
 		)
 	)
-	(hierarchical_label "Shift_Clock"
+	(hierarchical_label "clock_595"
 		(shape input)
 		(at 161.29 62.23 180)
@@
 		)
 	)
-	(hierarchical_label "no_en"
-		(shape input)
-		(at 161.29 72.39 180)
-		(effects
-			(font
-				(size 1.27 1.27)
-			)
-			(justify right)
-		)
-	)
 	(hierarchical_label "c3"
 		(shape input)
@@
 		)
 	)
-	(hierarchical_label "clock1_input"
+	(hierarchical_label "clock_165"
 		(shape input)
 		(at 91.44 82.55 180)
@@
 		)
 	)
-	(hierarchical_label "Storage_Clock"
+	(hierarchical_label "LATCH_595"
 		(shape input)
 		(at 161.29 69.85 180)
@@
 		)
 	)
-	(hierarchical_label "Parallel_Load"
+	(hierarchical_label "LOAD_165"
 		(shape input)
 		(at 91.44 77.47 180)
@@
 		)
 	)
-	(hierarchical_label "Row_Serial_H"
+	(hierarchical_label "DATA_OUT_165"
 		(shape input)
 		(at 116.84 52.07 0)
@@
 		(shape input)
 		(at 35.56 60.96 180)
-		(effects
-			(font
-				(size 1.27 1.27)
-			)
-			(justify right)
-		)
-	)
-	(hierarchical_label "Row_Serial_L"
-		(shape input)
-		(at 116.84 54.61 0)
-		(effects
-			(font
-				(size 1.27 1.27)
-			)
-			(justify left)
-		)
-	)
-	(hierarchical_label "Rst"
-		(shape input)
-		(at 161.29 64.77 180)
 		(effects
 			(font
@@
 			)
 		)
-		(property "Footprint" ""
+		(property "Footprint" "Package_SO:SOIC-16_3.9x9.9mm_P1.27mm"
 			(at 104.14 67.31 0)
 			(effects
@@
 			)
 		)
-		(property "Footprint" ""
+		(property "Footprint" "Connector_JST:JST_EH_B3B-EH-A_1x03_P2.50mm_Vertical"
 			(at 223.52 77.47 0)
 			(effects
@@
 			)
 		)
-		(property "Footprint" ""
+		(property "Footprint" "Connector_JST:JST_EH_B3B-EH-A_1x03_P2.50mm_Vertical"
 			(at 223.52 118.11 0)
 			(effects
@@
 			)
 		)
-		(property "Footprint" ""
+		(property "Footprint" "Connector_JST:JST_EH_B3B-EH-A_1x03_P2.50mm_Vertical"
 			(at 223.52 57.15 0)
 			(effects
@@
 	(symbol
 		(lib_id "power:+3.3V")
+		(at 161.29 64.77 90)
+		(unit 1)
+		(exclude_from_sim no)
+		(in_bom yes)
+		(on_board yes)
+		(dnp no)
+		(fields_autoplaced yes)
+		(property "Reference" "#PWR058"
+			(at 165.1 64.77 0)
+			(effects
+				(font
+					(size 1.27 1.27)
+				)
+				(hide yes)
+			)
+		)
+		(property "Value" "+3.3V"
+			(at 157.48 64.7699 90)
+			(effects
+				(font
+					(size 1.27 1.27)
+				)
+				(justify left)
+			)
+		)
+		(property "Footprint" ""
+			(at 161.29 64.77 0)
+			(effects
+				(font
+					(size 1.27 1.27)
+				)
+				(hide yes)
+			)
+		)
+		(property "Datasheet" ""
+			(at 161.29 64.77 0)
+			(effects
+				(font
+					(size 1.27 1.27)
+				)
+				(hide yes)
+			)
+		)
+		(property "Description" "Power symbol creates a global label with name \"+3.3V\""
+			(at 161.29 64.77 0)
+			(effects
+				(font
+					(size 1.27 1.27)
+				)
+				(hide yes)
+			)
+		)
+		(pin "1"
+		)
+		(instances
+			(project ""
+				(path "/473e845e-7ed3-42b5-aa14-5895a6f0c76b/87634a3e-a16c-4e1a-8724-f7b86e6a4f09"
+					(reference "#PWR058")
+					(unit 1)
+				)
+			)
+		)
+	)
+	(symbol
+		(lib_id "power:+3.3V")
 		(at 218.44 74.93 90)
 		(unit 1)
@@
 			)
 		)
-		(property "Footprint" ""
+		(property "Footprint" "Connector_JST:JST_EH_B3B-EH-A_1x03_P2.50mm_Vertical"
 			(at 223.52 107.95 0)
 			(effects
@@
 			)
 		)
-		(property "Footprint" ""
+		(property "Footprint" "Connector_JST:JST_EH_B3B-EH-A_1x03_P2.50mm_Vertical"
 			(at 223.52 67.31 0)
 			(effects
@@
 			)
 		)
-		(property "Footprint" ""
+		(property "Footprint" "Connector_JST:JST_EH_B7B-EH-A_1x07_P2.50mm_Vertical"
 			(at 40.64 63.5 0)
 			(effects
@@
 			)
 		)
-		(property "Footprint" ""
+		(property "Footprint" "Connector_JST:JST_EH_B3B-EH-A_1x03_P2.50mm_Vertical"
 			(at 223.52 87.63 0)
 			(effects
@@
 			)
 		)
-		(property "Footprint" ""
+		(property "Footprint" "Package_SO:SOIC-16_3.9x9.9mm_P1.27mm"
 			(at 171.45 67.31 0)
 			(effects
@@
 			)
 		)
-		(property "Footprint" ""
+		(property "Footprint" "Connector_JST:JST_EH_B3B-EH-A_1x03_P2.50mm_Vertical"
 			(at 223.52 97.79 0)
 			(effects
@@
 	(symbol
 		(lib_id "power:GND")
+		(at 161.29 72.39 270)
+		(unit 1)
+		(exclude_from_sim no)
+		(in_bom yes)
+		(on_board yes)
+		(dnp no)
+		(fields_autoplaced yes)
+		(property "Reference" "#PWR059"
+			(at 154.94 72.39 0)
+			(effects
+				(font
+					(size 1.27 1.27)
+				)
+				(hide yes)
+			)
+		)
+		(property "Value" "GND"
+			(at 157.48 72.3899 90)
+			(effects
+				(font
+					(size 1.27 1.27)
+				)
+				(justify right)
+			)
+		)
+		(property "Footprint" ""
+			(at 161.29 72.39 0)
+			(effects
+				(font
+					(size 1.27 1.27)
+				)
+				(hide yes)
+			)
+		)
+		(property "Datasheet" ""
+			(at 161.29 72.39 0)
+			(effects
+				(font
+					(size 1.27 1.27)
+				)
+				(hide yes)
+			)
+		)
+		(property "Description" "Power symbol creates a global label with name \"GND\" , ground"
+			(at 161.29 72.39 0)
+			(effects
+				(font
+					(size 1.27 1.27)
+				)
+				(hide yes)
+			)
+		)
+		(pin "1"
+		)
+		(instances
+			(project ""
+				(path "/473e845e-7ed3-42b5-aa14-5895a6f0c76b/87634a3e-a16c-4e1a-8724-f7b86e6a4f09"
+					(reference "#PWR059")
+					(unit 1)
+				)
+			)
+		)
+	)
+	(symbol
+		(lib_id "power:GND")
 		(at 91.44 72.39 270)
 		(unit 1)
@@
 					(unit 1)
 				)
+			)
+		)
+	)
+	(symbol
+		(lib_id "power:GND")
+		(at 171.45 85.09 0)
+		(unit 1)
+		(exclude_from_sim no)
+		(in_bom yes)
+		(on_board yes)
+		(dnp no)
+		(fields_autoplaced yes)
+		(property "Reference" "#PWR060"
+			(at 171.45 91.44 0)
+			(effects
+				(font
+					(size 1.27 1.27)
+				)
+				(hide yes)
+			)
+		)
+		(property "Value" "GND"
+			(at 171.45 90.17 0)
+			(effects
+				(font
+					(size 1.27 1.27)
+				)
+			)
+		)
+		(property "Footprint" ""
+			(at 171.45 85.09 0)
+			(effects
+				(font
+					(size 1.27 1.27)
+				)
+				(hide yes)
+			)
+		)
+		(property "Datasheet" ""
+			(at 171.45 85.09 0)
+			(effects
+				(font
+					(size 1.27 1.27)
+				)
+				(hide yes)
+			)
+		)
+		(property "Description" "Power symbol creates a global label with name \"GND\" , ground"
+			(at 171.45 85.09 0)
+			(effects
+				(font
+					(size 1.27 1.27)
+				)
+				(hide yes)
+			)
+		)
+		(pin "1"
+		)
+		(instances
+			(project ""
+				(path "/473e845e-7ed3-42b5-aa14-5895a6f0c76b/87634a3e-a16c-4e1a-8724-f7b86e6a4f09"
+					(reference "#PWR060")
+					(unit 1)
+				)

Commit message: more pcb edit
Parts:
- added J14: Jack-DC, Connector_Audio:Jack_3.5mm_CUI_SJ-3523-SMT_Horizontal, symbol Connector:Jack-DC
- added J4: DIN-5, Connector_JST:JST_EH_B2B-EH-A_1x02_P2.50mm_Vertical, symbol Connector:DIN-5
- added R29, R30, R31: 330, Resistor_SMD:R_0402_1005Metric, symbol Device:R_Small
- added U4: 6N138, Package_DIP:DIP-8_W7.62mm_LongPads, symbol Isolator:6N138
- J5: symbol Connector:Conn_01x07_Socket -> Connector:Conn_01x10_Socket
Connections:
- net +3.3V: now also R30.1, U4.8 (VCC)
- net GND: now also U4.3 (C2), U4.5 (GND)
- net jst0: no longer J5.1 (Pin_1)
- new net: J4.4, R31.1
- new net: J14.2, R31.2, U4.7 (VO1)
- new net: J14.1, J4.5, R30.2, U4.6 (VO2)
- new net: R29.2, U4.2 (C1)
- new net midi_in: R29.1
- no-connect marks 1 -> 4
