File: Hardware/PCB_CAD/MuseMatrix_Core/Raspberry_connections.kicad_sch (KiCad schematic)
At the start: 1 part, among them J1 Raspberry_Pi_4

Commit message: more pcb edit
Parts:
- J1: footprint (none) -> Connector_PinHeader_1.00mm:PinHeader_2x16_P1.00mm_Vertical
Connections:
- net data_595: now reaches J1.11 (GPIO17/SPI1_~{CE1})
- net clock_595: now reaches J1.13 (GPIO27/SDIO_DAT3)
- net latch_595: now reaches J1.15 (GPIO22/SDIO_CLK)
- net parallel_load_165: now reaches J1.16 (GPIO23/SDIO_CMD)
- net Clock_165: now reaches J1.18 (GPIO24/SDIO_DAT0)
- net ADC_data_in: now reaches J1.19 (MOSI_SPI0/GPIO10)
- net ADC_data_out: now reaches J1.21 (MISO_SPI0/GPIO09)
- net Serial_out_165: now reaches J1.22 (GPIO25/SDIO_DAT1)
- net ADC_clock: now reaches J1.23 (SCLK_SPI0/GPIO11)
- net ADC_select: now reaches J1.24 (~{CE0}_SPI0/GPIO08)
- net midi_out: now reaches J1.8 (GPIO14/UART_TXD)
- net 5V: no longer names the net of J1.2 (5V), J1.4 (5V)
- net I2C_SCL: no longer names the net of J1.5 (SCL_I2C1/GPIO03)
- net I2C_SDA: no longer names the net of J1.3 (SDA_I2C1/GPIO02)
- no-connect marks 0 -> 1
Changed lines of the file:
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@@
 	(generator_version "8.0")
 	(paper "A4")
-	(hierarchical_label "5V"
+	(no_connect
+		(at 168.91 53.34)
+	)
+	(hierarchical_label "ADC_data_out"
 		(shape input)
-		(at 168.91 53.34 0)
+		(at 168.91 91.44 0)
+		(effects
+			(font
+				(size 1.27 1.27)
+			)
+			(justify left)
+		)
+	)
+	(hierarchical_label "ADC_select"
+		(shape input)
+		(at 168.91 88.9 0)
+		(effects
+			(font
+				(size 1.27 1.27)
+			)
+			(justify left)
+		)
+	)
+	(hierarchical_label "ADC_data_in"
+		(shape input)
+		(at 168.91 93.98 0)
 		(effects
 			(font
@@
 		)
 	)
-	(hierarchical_label "I2C_SDA"
+	(hierarchical_label "clock_595"
 		(shape input)
-		(at 168.91 68.58 0)
+		(at 102.87 99.06 180)
+		(effects
+			(font
+				(size 1.27 1.27)
+			)
+			(justify right)
+		)
+	)
+	(hierarchical_label "ADC_clock"
+		(shape input)
+		(at 168.91 96.52 0)
 		(effects
 			(font
@@
 		)
 	)
-	(hierarchical_label "I2C_SCL"
+	(hierarchical_label "midi_out"
 		(shape input)
-		(at 168.91 71.12 0)
+		(at 102.87 60.96 180)
 		(effects
 			(font
 				(size 1.27 1.27)
 			)
-			(justify left)
+			(justify right)
+		)
+	)
+	(hierarchical_label "data_595"
+		(shape input)
+		(at 102.87 71.12 180)
+		(effects
+			(font
+				(size 1.27 1.27)
+			)
+			(justify right)
+		)
+	)
+	(hierarchical_label "Clock_165"
+		(shape input)
+		(at 102.87 91.44 180)
+		(effects
+			(font
+				(size 1.27 1.27)
+			)
+			(justify right)
+		)
+	)
+	(hierarchical_label "parallel_load_165"
+		(shape input)
+		(at 102.87 88.9 180)
+		(effects
+			(font
+				(size 1.27 1.27)
+			)
+			(justify right)
+		)
+	)
+	(hierarchical_label "Serial_out_165"
+		(shape input)
+		(at 102.87 93.98 180)
+		(effects
+			(font
+				(size 1.27 1.27)
+			)
+			(justify right)
+		)
+	)
+	(hierarchical_label "latch_595"
+		(shape input)
+		(at 102.87 86.36 180)
+		(effects
+			(font
+				(size 1.27 1.27)
+			)
+			(justify right)
 		)
 	)
@@
 			)
 		)
-		(property "Footprint" ""
+		(property "Footprint" "Connector_PinHeader_1.00mm:PinHeader_2x16_P1.00mm_Vertical"
 			(at 205.994 123.698 0)
 			(effects
