File: Hardware/PCB_CAD/MuseMatrix_Core/Raspberry_connections.kicad_sch (KiCad schematic)
At the start: 1 part, among them J1 Raspberry_Pi_4

Commit message: update
Connections:
- no-connect marks 1 -> 18
Changed lines of the file:
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@@
+	)
+	(no_connect
+		(at 168.91 76.2)
+	)
+	(no_connect
+		(at 168.91 78.74)
+	)
+	(no_connect
+		(at 102.87 73.66)
+	)
+	(no_connect
+		(at 102.87 76.2)
+	)
+	(no_connect
+		(at 168.91 86.36)
+	)
+	(no_connect
+		(at 102.87 68.58)
 	)
 	(no_connect
 		(at 168.91 53.34)
 	)
+	(no_connect
+		(at 168.91 63.5)
+	)
+	(no_connect
+		(at 168.91 68.58)
+	)
+	(no_connect
+		(at 102.87 78.74)
+	)
+	(no_connect
+		(at 102.87 81.28)
+	)
+	(no_connect
+		(at 168.91 71.12)
+	)
+	(no_connect
+		(at 102.87 55.88)
+	)
+	(no_connect
+		(at 102.87 96.52)
+	)
+	(no_connect
+		(at 168.91 60.96)
+	)
+	(no_connect
+		(at 102.87 53.34)
+	)
+	(no_connect
+		(at 102.87 63.5)
+	)
+	(no_connect
+		(at 168.91 81.28)
+	)
 	(wire

Commit message: separated in 2 boards
Parts:
- J1: footprint Connector_PinHeader_1.00mm:PinHeader_2x16_P1.00mm_Vertical -> Connector_PinHeader_2.54mm:PinHeader_1x16_P2.54mm_Vertical
Changed lines of the file:
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@@
 		(shape input)
 		(at 168.91 91.44 0)
-		(fields_autoplaced yes)
 		(effects
 			(font
@@
 		(shape input)
 		(at 168.91 88.9 0)
-		(fields_autoplaced yes)
 		(effects
 			(font
@@
 		(shape input)
 		(at 168.91 93.98 0)
-		(fields_autoplaced yes)
 		(effects
 			(font
@@
 		(shape input)
 		(at 135.89 104.14 270)
-		(fields_autoplaced yes)
 		(effects
 			(font
@@
 		(shape input)
 		(at 102.87 99.06 180)
-		(fields_autoplaced yes)
 		(effects
 			(font
@@
 		(shape input)
 		(at 168.91 96.52 0)
-		(fields_autoplaced yes)
 		(effects
 			(font
@@
 		(shape input)
 		(at 175.26 53.34 0)
-		(fields_autoplaced yes)
 		(effects
 			(font
@@
 		(shape input)
 		(at 102.87 60.96 180)
-		(fields_autoplaced yes)
 		(effects
 			(font
@@
 		(shape input)
 		(at 102.87 71.12 180)
-		(fields_autoplaced yes)
 		(effects
 			(font
@@
 		(shape input)
 		(at 102.87 91.44 180)
-		(fields_autoplaced yes)
 		(effects
 			(font
@@
 		(shape input)
 		(at 102.87 88.9 180)
-		(fields_autoplaced yes)
 		(effects
 			(font
@@
 		(shape input)
 		(at 102.87 93.98 180)
-		(fields_autoplaced yes)
 		(effects
 			(font
@@
 		(shape input)
 		(at 102.87 86.36 180)
-		(fields_autoplaced yes)
 		(effects
 			(font
@@
 			)
 		)
-		(property "Footprint" "Connector_PinHeader_1.00mm:PinHeader_2x16_P1.00mm_Vertical"
+		(property "Footprint" "Connector_PinHeader_2.54mm:PinHeader_1x16_P2.54mm_Vertical"
 			(at 205.994 123.698 0)
 			(effects
