File: Hardware/PCB_CAD/MuseMatrix_Core/MuseMatrix_Core.kicad_sch (KiCad schematic)
At the start: 0 parts

Commit message: pcb update
Other:
- added sheet Octaves board (octaves.kicad_sch)
Changed lines of the file:
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@@
 	(paper "A4")
+	(sheet
+		(at 214.3 31.6)
+		(size 48.8 27.9)
+		(fields_autoplaced yes)
+		(stroke
+			(width 0.1524)
+			(type solid)
+		)
+		(fill
+			(color 0 0 0 0.0000)
+		)
+		(property "Sheetname" "Octaves board"
+			(at 214.3 30.8884 0)
+			(effects
+				(font
+					(size 1.27 1.27)
+				)
+				(justify left bottom)
+			)
+		)
+		(property "Sheetfile" "octaves.kicad_sch"
+			(at 214.3 60.0846 0)
+			(effects
+				(font
+					(size 1.27 1.27)
+				)
+				(justify left top)
+			)
+		)
+		(instances
+			(project "MuseMatrix_Core"
+				(path "/473e845e-7ed3-42b5-aa14-5895a6f0c76b"
+					(page "6")
+				)
+			)
+		)
+	)
 	(sheet
 		(at 132.2 24.7)

Commit message: more pcb edit
Other:
- sheet Column_7_Rows ports: added 3.3V, Column_voltage; removed none
- sheet Main_board ports: added DATA_IN_595, DATA_OUT_165, LATCH_595, LOAD_165, clock_165, clock_595, midi_in; removed Parallel_Load, Row_Serial_H, Row_Serial_L, Rst, Serial_Column_input, Shift_Clock, Storage_Clock, clock1_input, no_en
- sheet Octaves board ports: added ADC_clock, DATA_IN_ADC, DATA_OUT_ADC, select; removed none
- sheet Raspberry_connections ports: added ADC_clock, ADC_data_in, ADC_data_out, ADC_select, Clock_165, Serial_out_165, clock_595, data_595, latch_595, midi_out, parallel_load_165; removed I2C_SCL, I2C_SDA
