File: Hardware/PCB_CAD/MuseMatrix_Core/octaves.kicad_sch (KiCad schematic)
At the start: 9 parts, among them U1 MCP3008

Commit message: more pcb edit
Connections:
- net select: now reaches U1.10 (~{CS}/SHDN)
- net ADC_clock: now reaches U1.13 (CLK)
Changed lines of the file:
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@@
+		)
+	)
+	(hierarchical_label "ADC_clock"
+		(shape input)
+		(at 212.09 95.25 0)
+		(effects
+			(font
+				(size 1.27 1.27)
+			)
+			(justify left)
 		)
 	)
@@
 		(effects
 			(font
+				(size 1.27 1.27)
+			)
+			(justify left)
+		)
+	)
+	(hierarchical_label "select"
+		(shape input)
+		(at 212.09 102.87 0)
+		(effects
+			(font
